Commit message: Parte 2

File: src/mi_robot_mecanum/urdf/mi_robot.urdf.xacro (robot description, xacro)
@@ -60,4 +60,5 @@
       </collision>
     <inertial>
+      <mass value="${rueda_masa}"/>
       <xacro:inercia_cilindro m="${rueda_masa}" r="${rueda_radio}" h="${rueda_ancho}"/>
     </inertial>
@@ -67,6 +68,6 @@
       <parent link="base_link"/>
       <child link="rueda_${prefijo}"/>
-      <origin xyz="${x_signo*lx} ${y_signo*ly} 0" rpy="0 0 0"/>
-      <axis xyz="0 1 0"/>
+      <origin xyz="${x_signo*lx} ${y_signo*ly} 0" rpy="${-pi/2} 0 0"/>
+      <axis xyz="0 0 1"/>
     </joint>
     <!-- TODO: joint "joint_rueda_${prefijo}" tipo continuous entre base_link y
@@ -82,18 +83,15 @@
   <!-- TODO: link "lidar_link" (cilindro) con dimensiones y masa de la hoja de datos:
        visual, collision e inertial -->
-  <link name="lindar_link">
+  <link name="lidar_link">
     <visual>
-      <origin xyz="0 0 0.14" rpy="0 0 0"/>
-      <geometry><cylindezr radius="0.039" length="0.041" /></geometry>
-      <material name="azul"><color rgba="0.2 0.4 0.8 1"/></material>
+      <geometry><cylinder radius="0.038" length="0.041" /></geometry>
+      <material name="negro"/>
     </visual>
     <collision>
-      <origin xyz="0 0 0.14" rpy="0 0 0"/>
-      <geometry><sphere radius="0.039"/></geometry>
+      <geometry><cylinder radius="0.038" length="0.041"/></geometry>
     </collision>
     <inertial>
-      <origin xyz="0 0 0.14" rpy="0 0 0"/>
       <mass value="0.190"/>
-      <xacro:inercia_cilindro m="0.190" r="0.039" h="0.041"/>
+      <xacro:inercia_cilindro m="0.190" r="0.038" h="0.041"/>
     </inertial>
   </link>
@@ -102,5 +100,5 @@
   <parent link="base_link"/>
   <child link="lidar_link"/>
-  <origin xyz="0.0 0 0.14" rpy="${-pi/2} 0 ${-pi/2}"/>
+  <origin xyz="0.0 0 0.14" rpy="0 0 0"/>
   </joint>
   <gazebo reference="lidar_link">
@@ -138,16 +136,13 @@
   <link name="camara_link">
     <visual>
-      <origin xyz="0.14 0 0.08" rpy="0 0 0"/>
-      <geometry><box size="0.165 0.048 0.040"/></geometry>
-      <material name="azul"><color rgba="0.2 0.4 0.8 1"/></material>
+      <geometry><box size="0.040 0.165 0.048"/></geometry>
+      <material name="negro"/>
     </visual>
     <collision>
-      <origin xyz="0.14 0 0.08" rpy="0 0 0"/>
-      <geometry><box size="0.165 0.048 0.040"/></geometry>
+      <geometry><box size="0.040 0.165 0.048"/></geometry>
     </collision>
     <inertial>
-      <origin xyz="0.14 0 0.08" rpy="0 0 0"/>
       <mass value="0.310"/>
-      <xacro:inercia_caja m="0.310" x="0.165" y="0.048" z="0.040"/>
+      <xacro:inercia_caja m="0.310" x="0.040" y="0.165" z="0.048"/>
     </inertial>
   </link>
@@ -160,12 +155,18 @@
   <!-- TODO: link "camara_optica_link" y joint fijo "joint_camara_optica" desde
        camara_link con rpy = (-π/2, 0, -π/2) (REP-103) -->
+  <link name="camara_optica_link"/>
+  <joint name="joint_camara_optica" type="fixed">
+    <parent link="camara_link"/>
+    <child link="camara_optica_link"/>
+    <origin xyz="0 0 0" rpy="${-pi/2} 0 ${-pi/2}"/>
+  </joint>
   <gazebo reference="camara_link">
     <sensor name="astra" type="rgbd_camera">
       <topic>/camara</topic>
-      <gz_frame_id>camera_optical_link</gz_frame_id>
+      <gz_frame_id>camara_optica_link</gz_frame_id>
       <update_rate>30</update_rate>
       <always_on>1</always_on>
       <camera>
-        <horizontal_fov>1,012291</horizontal_fov>   <!-- en radianes -->
+        <horizontal_fov>${58.4*pi/180}</horizontal_fov>   <!-- en radianes -->
         <image>
           <width>640</width>
